File: [Hardware]/100008_hw-vern-aqm/100008_hw-vern-aqm.kicad_sch (KiCad schematic)
At the start: 0 parts

Commit message: end of day work
Other:
- removed sheet Power - Sequencing
Changed lines of the file:
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@@
-	)
-	(sheet
-		(at 340.36 313.69)
-		(size 35.56 5.08)
-		(stroke
-			(width 0.1524)
-			(type solid)
-		)
-		(fill
-			(color 0 0 0 0.0000)
-		)
-		(property "Sheetname" "Power - Sequencing"
-			(at 340.36 312.6609 0)
-			(effects
-				(font
-					(face "Times New Roman")
-					(size 1.905 1.905)
-					(bold yes)
-					(color 0 0 0 1)
-				)
-				(justify left bottom)
-			)
-		)
-		(property "Sheetfile" "Power - Sequencing.kicad_sch"
-			(at 341.63 314.96 0)
-			(effects
-				(font
-					(face "Arial")
-					(size 1.27 1.27)
-				)
-				(justify left top)
-			)
-		)
-		(instances
-			(project "100008_hw-vern-aqm"
-				(path "/0650c7a8-acba-429c-9f8e-eec0baf0bc1c"
-					(page "6")
-				)
-			)
-		)
 	)
 	(sheet

Commit message: mid day progress
Other:
- note added: "Connectors and Power"
- note added: "MCU - ESP32"
- note added: "Sensors"
- note removed: "Power - Sequencing"
- note removed: "Random Sheet 1"
- note removed: "Random Sheet 2"
Changed lines of the file:
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@@
 		)
 	)
-	(text "Random Sheet 1"
+	(text "Connectors and Power"
 		(exclude_from_sim no)
 		(at 45.72 106.68 0)
@@
 		)
 	)
-	(text "Random Sheet 2"
+	(text "MCU - ESP32"
 		(exclude_from_sim no)
 		(at 45.72 114.3 0)
@@
 		)
 	)
-	(text "Power - Sequencing"
+	(text "Sensors"
 		(exclude_from_sim no)
 		(at 45.72 121.92 0)
