File: [Hardware]/100008_hw-vern-aqm/sensors.kicad_sch (KiCad schematic)
At the start: 7 parts

Commit message: end of day work
Parts:
- removed SW? (x2): SW_Push, symbol Switch:SW_Push
- removed U?: ESP32-S3-WROOM-1, PCM_Espressif:ESP32-S3-WROOM-1, symbol PCM_Espressif:ESP32-S3-WROOM-1
- added U?: SCD40-D-R2, Sensor:Sensirion_SCD4x-1EP_10.1x10.1mm_P1.25mm_EP4.8x4.8mm, symbol Sensor_Gas:SCD40-D-R2
Connections:
- new net: U?.19 (VDD), U?.7 (VDD)
- new net: U?.20 (GND), U?.21 (GND), U?.6 (GND)
Other:
- moved on the sheet: C?, R?

Commit message: mid day progress
Other:
- title: MCU - ESP32 -> Sensors
Changed lines of the file:
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@@
 	(paper "A3")
 	(title_block
-		(title "MCU - ESP32")
+		(title "Sensors")
 		(date "Last Modified Date")
 		(rev "${REVISION}")
