File: Hardware/100008_hw-vern-aqm/Project Architecture.kicad_sch (KiCad schematic)
At the start: 0 parts

Commit message: schematic work
Changed lines of the file:
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@@
 	(polyline
 		(pts
-			(xy 195.58 58.42) (xy 195.58 69.85)
-		)
-		(stroke
-			(width 0)
-			(type default)
-		)
-	)
-	(polyline
-		(pts
-			(xy 195.58 55.88) (xy 195.58 44.45)
+			(xy 243.84 55.88) (xy 243.84 44.45)
+		)
+		(stroke
+			(width 0)
+			(type default)
+		)
+	)
+	(polyline
+		(pts
+			(xy 243.84 58.42) (xy 243.84 69.85)
 		)
 		(stroke
@@
 		(pts
 			(xy 243.84 85.09) (xy 243.84 93.98)
+		)
+		(stroke
+			(width 0)
+			(type default)
+		)
+	)
+	(polyline
+		(pts
+			(xy 243.84 133.35) (xy 243.84 142.24)
+		)
+		(stroke
+			(width 0)
+			(type default)
+		)
+	)
+	(polyline
+		(pts
+			(xy 243.84 121.92) (xy 243.84 130.81)
 		)
 		(stroke
@@
 	)
 	(arc
-		(start 195.58 55.88)
-		(mid 195.2051 56.7751)
-		(end 194.31 57.15)
+		(start 245.13 132.06)
+		(mid 244.2349 131.6851)
+		(end 243.86 130.79)
+		(stroke
+			(width 0)
+			(type default)
+		)
+		(fill
+			(type none)
+		)
+	)
+	(arc
+		(start 243.84 58.42)
+		(mid 244.2149 57.5249)
+		(end 245.11 57.15)
 		(stroke
 			(width 0)
@@
 	)
 	(arc
-		(start 194.31 57.15)
-		(mid 195.2051 57.5249)
-		(end 195.58 58.42)
+		(start 245.11 57.15)
+		(mid 244.2149 56.7751)
+		(end 243.84 55.88)
+		(stroke
+			(width 0)
+			(type default)
+		)
+		(fill
+			(type none)
+		)
+	)
+	(arc
+		(start 243.86 142.22)
+		(mid 243.1161 144.0161)
+		(end 241.32 144.76)
 		(stroke
 			(width 0)
@@
 	)
 	(arc
-		(start 195.58 44.45)
-		(mid 196.3239 42.6539)
-		(end 198.12 41.91)
-		(stroke
-			(width 0)
-			(type default)
-		)
-		(fill
-			(type none)
-		)
-	)
-	(arc
-		(start 198.12 72.39)
-		(mid 196.3298 71.6402)
-		(end 195.58 69.85)
-		(stroke
-			(width 0)
-			(type default)
-		)
-		(fill
-			(type none)
-		)
-	)
-	(text_box "Description"
-		(exclude_from_sim no)
-		(at 176.53 54.61 0)
-		(size 17.145 5.08)
+		(start 243.84 69.85)
+		(mid 243.0961 71.6461)
+		(end 241.3 72.39)
+		(stroke
+			(width 0)
+			(type default)
+		)
+		(fill
+			(type none)
+		)
+	)
+	(arc
+		(start 241.3 41.91)
+		(mid 243.0902 42.6598)
+		(end 243.84 44.45)
+		(stroke
+			(width 0)
+			(type default)
+		)
+		(fill
+			(type none)
+		)
+	)
+	(arc
+		(start 241.32 119.36)
+		(mid 243.1102 120.1098)
+		(end 243.86 121.9)
+		(stroke
+			(width 0)
+			(type default)
+		)
+		(fill
+			(type none)
+		)
+	)
+	(arc
+		(start 243.86 133.33)
+		(mid 244.2349 132.4349)
+		(end 245.13 132.06)
+		(stroke
+			(width 0)
+			(type default)
+		)
+		(fill
+			(type none)
+		)
+	)
+	(text_box "USB, Debug and Sensor connectors and Power Supply"
+		(exclude_from_sim no)
+		(at 246.38 54.61 0)
+		(size 33.02 12.7)
 		(stroke
 			(width -0.0001)
@@
 				(color 0 0 0 1)
 			)
-			(justify right top)
+			(justify left top)
 		)
 	)
@@
 		)
 	)
-	(text_box "Description"
+	(text_box "CO2 and Pressure Sensors"
+		(exclude_from_sim no)
+		(at 245.11 129.54 0)
+		(size 29.21 10.16)
+		(stroke
+			(width -0.0001)
+			(type default)
+		)
+		(fill
+			(type none)
+		)
+		(effects
+			(font
+				(size 1.905 1.905)
+				(thickness 0.381)
+				(bold yes)
+				(color 0 0 0 1)
+			)
+			(justify left top)
+		)
+	)
+	(text_box "Microcontroller"
 		(exclude_from_sim no)
 		(at 245.11 92.71 0)
@@
 			(project "100008_hw-vern-aqm"
 				(path "/0650c7a8-acba-429c-9f8e-eec0baf0bc1c/fede4c36-00cc-4d3d-b71c-5243ba232202"
-					(page "4")
+					(page "3")
 				)
 			)
@@
 			(project "100008_hw-vern-aqm"
 				(path "/0650c7a8-acba-429c-9f8e-eec0baf0bc1c/fede4c36-00cc-4d3d-b71c-5243ba232202"
-					(page "6")
+					(page "5")
 				)
 			)
@@
 			(project "100008_hw-vern-aqm"
 				(path "/0650c7a8-acba-429c-9f8e-eec0baf0bc1c/fede4c36-00cc-4d3d-b71c-5243ba232202"
-					(page "5")
-				)
-			)
+					(page "4")
+				)
+			)
