File: Hardware/100008_hw-vern-aqm/_autosave-connectors-and-power.kicad_sch (KiCad schematic)
At the start: 41 parts, among them J1 Conn_01x14_Socket, J2 USB4220-03-1000-C, J3 Conn_01x06_MountingPin, J4 Conn_01x03_Pin, J5 Conn_01x06_Socket, J6 Conn_01x04_Socket, J7 Conn_01x05_Pin, U1 AMS1117-3.3

Commit message: pcb routing
Parts:
- gave numbers to parts that had none: 1
Changed lines of the file:
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@@
 		(on_board yes)
 		(dnp yes)
-		(property "Reference" "J?"
+		(property "Reference" "J8"
 			(at 275.59 172.72 0)
 			(effects
@@
 			(project ""
 				(path "/0650c7a8-acba-429c-9f8e-eec0baf0bc1c/fede4c36-00cc-4d3d-b71c-5243ba232202/7d5a1283-086b-46b0-8df7-a9850521fb5e"
-					(reference "J?")
+					(reference "J8")
 					(unit 1)
 				)
