File: Hardware/100008_hw-vern-aqm/mcu-esp32.kicad_sch (KiCad schematic)
At the start: 7 parts

Commit message: renamed folders
Connections:
- net GND: now also SW?.2, SW?.2
- net GPIO0: now also SW?.1
- net RESET: now reaches C?.1, R?.2, U?.3 (EN)
- net RESET: now also SW?.1
- no-connect marks 0 -> 3
Other:
- note added: "Reset and GPIO0 buttons"
- moved on the sheet: C?, R?, SW?

Commit message: schematic work
Parts:
- added C?: 10u, Capacitor_SMD:C_0805_2012Metric, symbol Device:C
- added C?: 100n, Capacitor_SMD:C_0603_1608Metric, symbol Device:C
- added R? (x2): 0R0, Resistor_SMD:R_0603_1608Metric, symbol Device:R
- added U?: CP2102N-Axx-xQFN24, Package_DFN_QFN:QFN-24-1EP_4x4mm_P0.5mm_EP2.6x2.6mm, symbol Interface_USB:CP2102N-Axx-xQFN24
Connections:
- net GND: now also C?.2, C?.2
- net USB_D+: now also R?.2
- net USB_D-: now also R?.2
- new net: R?.1, U?.3 (D+)
- new net: R?.1, U?.4 (D-)
- new net: U?.2 (GND), U?.25 (GND)
- new net VBUS: C?.1, C?.1, U?.8 (VBUS)
Other:
- moved on the sheet: C?, R?, SW?, U?

Commit message: schematic work
Parts:
- removed C?: 1u, Capacitor_SMD:C_0805_2012Metric, symbol Device:C
- removed SW?: SW_Push, symbol Switch:SW_Push
- added C? (x3): 100n, Capacitor_SMD:C_0603_1608Metric, symbol Device:C
- added SW?: SW_Push, Button_Switch_SMD:SW_Tactile_SPST_NO_Straight_CK_PTS636Sx25SMTRLFS, symbol Switch:SW_Push
- SW?: footprint (none) -> Button_Switch_SMD:SW_Tactile_SPST_NO_Straight_CK_PTS636Sx25SMTRLFS; MFN (none) -> PTS636 SK25 SMTR LFS
Connections:
- net GND: now also C?.2, C?.2, C?.2, SW?.2
- net GPIO0: now also C?.1
- net RESET: now also C?.1, C?.1, SW?.1
Other:
- moved on the sheet: SW?

Commit message: schematic and pcb work
Changed lines of the file:
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@@
 	(wire
 		(pts
-			(xy 203.2 93.98) (xy 217.17 93.98)
+			(xy 203.2 93.98) (xy 215.9 93.98)
 		)
 		(stroke
@@
 	(wire
 		(pts
+			(xy 210.82 153.67) (xy 231.14 153.67)
+		)
+		(stroke
+			(width 0)
+			(type default)
+		)
+	)
+	(wire
+		(pts
 			(xy 123.19 185.42) (xy 125.73 185.42)
 		)
@@
 	(wire
 		(pts
+			(xy 210.82 158.75) (xy 231.14 158.75)
+		)
+		(stroke
+			(width 0)
+			(type default)
+		)
+	)
+	(wire
+		(pts
 			(xy 293.37 120.65) (xy 299.72 120.65)
 		)
@@
 		(pts
 			(xy 91.44 78.74) (xy 111.76 78.74)
+		)
+		(stroke
+			(width 0)
+			(type default)
+		)
+	)
+	(wire
+		(pts
+			(xy 210.82 151.13) (xy 231.14 151.13)
+		)
+		(stroke
+			(width 0)
+			(type default)
+		)
+	)
+	(wire
+		(pts
+			(xy 210.82 156.21) (xy 231.14 156.21)
 		)
 		(stroke
@@
 	)
 	(label "GPIO0"
-		(at 217.17 93.98 180)
+		(at 215.9 93.98 180)
 		(fields_autoplaced yes)
 		(effects
@@
 		)
 	)
+	(label "SD_SCK(CLK)"
+		(at 212.09 158.75 0)
+		(fields_autoplaced yes)
+		(effects
+			(font
+				(size 1.27 1.27)
+			)
+			(justify left bottom)
+		)
+	)
 	(label "SPI_MISO"
 		(at 212.09 127 0)
@@
 		)
 	)
+	(label "SD_MOSI(CMD)"
+		(at 212.09 153.67 0)
+		(fields_autoplaced yes)
+		(effects
+			(font
+				(size 1.27 1.27)
+			)
+			(justify left bottom)
+		)
+	)
 	(label "SPI_nCS_TOUCH"
 		(at 212.09 114.3 0)
@@
 			)
 			(justify right bottom)
+		)
+	)
+	(label "SD_CS(D3)"
+		(at 212.09 151.13 0)
+		(fields_autoplaced yes)
+		(effects
+			(font
+				(size 1.27 1.27)
+			)
+			(justify left bottom)
+		)
+	)
+	(label "SD_MISO(D0)"
+		(at 212.09 156.21 0)
+		(fields_autoplaced yes)
+		(effects
+			(font
+				(size 1.27 1.27)
+			)
+			(justify left bottom)
 		)
 	)
@@
 		)
 	)
+	(global_label "SD_CS(D3)"
+		(shape bidirectional)
+		(at 231.14 151.13 0)
+		(fields_autoplaced yes)
+		(effects
+			(font
+				(size 1.27 1.27)
+			)
+			(justify left)
+		)
+		(property "Intersheetrefs" "${INTERSHEET_REFS}"
+			(at 245.336 151.13 0)
+			(effects
+				(font
+					(size 1.27 1.27)
+				)
+				(justify left)
+				(hide yes)
+			)
+		)
+	)
 	(global_label "USB_D+"
 		(shape bidirectional)
@@
 		)
 	)
+	(global_label "SD_MISO(D0)"
+		(shape bidirectional)
+		(at 231.14 156.21 0)
+		(fields_autoplaced yes)
+		(effects
+			(font
+				(size 1.27 1.27)
+			)
+			(justify left)
+		)
+		(property "Intersheetrefs" "${INTERSHEET_REFS}"
+			(at 247.4527 156.21 0)
+			(effects
+				(font
+					(size 1.27 1.27)
+				)
+				(justify left)
+				(hide yes)
+			)
+		)
+	)
 	(global_label "SPI_SCK"
 		(shape input)
@@
 		)
 	)
+	(global_label "SD_SCK(CLK)"
+		(shape bidirectional)
+		(at 231.14 158.75 0)
+		(fields_autoplaced yes)
+		(effects
+			(font
+				(size 1.27 1.27)
+			)
+			(justify left)
+		)
+		(property "Intersheetrefs" "${INTERSHEET_REFS}"
+			(at 247.6946 158.75 0)
+			(effects
+				(font
+					(size 1.27 1.27)
+				)
+				(justify left)
+				(hide yes)
+			)
+		)
+	)
 	(global_label "I2C_SDA"
 		(shape bidirectional)
@@
 		(property "Intersheetrefs" "${INTERSHEET_REFS}"
 			(at 245.0713 111.76 0)
+			(effects
+				(font
+					(size 1.27 1.27)
+				)
+				(justify left)
+				(hide yes)
+			)
+		)
+	)
+	(global_label "SD_MOSI(CMD)"
+		(shape bidirectional)
+		(at 231.14 153.67 0)
+		(fields_autoplaced yes)
+		(effects
+			(font
+				(size 1.27 1.27)
+			)
+			(justify left)
+		)
+		(property "Intersheetrefs" "${INTERSHEET_REFS}"
+			(at 248.9646 153.67 0)
 			(effects
 				(font
@@
 		)
 		(instances
-			(project ""
+			(project "100008_hw-vern-aqm"
 				(path "/0650c7a8-acba-429c-9f8e-eec0baf0bc1c/fede4c36-00cc-4d3d-b71c-5243ba232202/e6015f1e-cbce-46f4-85e1-3d5463a17dc1"
 					(reference "U?")

Commit message: schematic and pcb layout
Parts:
- added C10: 10u, Capacitor_SMD:C_0805_2012Metric, symbol Device:C
- added C13: 100n, Capacitor_SMD:C_0603_1608Metric, symbol Device:C
- added D8, D9: LED, LED_SMD:LED_0603_1608Metric, symbol Device:LED
- added Q1, Q2: BC817, Package_TO_SOT_SMD:SOT-23, symbol Transistor_BJT:BC817
- added R18: 5k1, Resistor_SMD:R_0603_1608Metric, symbol Device:R
- added R19, R23, R24, R27: 10k, Resistor_SMD:R_0603_1608Metric, symbol Device:R
- added R20, R28, R29: 1k, Resistor_SMD:R_0603_1608Metric, symbol Device:R
- added R25, R26, R30, R31: 0R0, Resistor_SMD:R_0603_1608Metric, symbol Device:R
- gave numbers to parts that had none: 14
Connections:
- net +3V3: now also C14.1, C15.1, U3.5 (VIO), U3.6 (VDD), U3.7 (VREGIN), C10.1, D8.2 (A), D9.2 (A), R20.1
- net GND: now also U3.2 (GND), U3.25 (GND), C10.2, C13.2, R19.2, R27.2
- net GPIO0: now also R31.1
- net I2C_SCL: now also U2.38 (GPIO2/TOUCH2/ADC1_CH1)
- net I2C_SDA: now also U2.39 (GPIO1/TOUCH1/ADC1_CH0)
- net LCD_BACKLIGHT: now also U2.19 (GPIO11/TOUCH11/ADC2_CH0/FSPID/FSPIIO5/SUBSPID)
- net LCD_DC/RS: now also U2.18 (GPIO10/TOUCH10/ADC1_CH9/FSPICS0/FSPIIO4/SUBSPICS0)
- net LCD_RESET: now also U2.17 (GPIO9/TOUCH9/ADC1_CH8/FSPIHD/SUBSPIHD)
- net RESET: now also R30.1
- net SD_CS(D3): now also U2.20 (GPIO12/TOUCH12/ADC2_CH1/FSPICLK/FSPIIO6/SUBSPICLK)
- net SD_MISO(D0): now also U2.22 (GPIO14/TOUCH14/ADC2_CH3/FSPIWP/FSPIDQS/SUBSPIWP)
- net SD_MOSI(CMD): now also U2.21 (GPIO13/TOUCH13/ADC2_CH2/FSPIQ/FSPIIO7/SUBSPIQ)
- net SD_SCK(CLK): now also U2.10 (GPIO17/U1TXD/ADC2_CH6)
- net SPI_MISO: now also U2.6 (GPIO6/TOUCH6/ADC1_CH5)
- net SPI_MOSI: now also U2.7 (GPIO7/TOUCH7/ADC1_CH6)
- net SPI_SCK: now also U2.12 (GPIO8/TOUCH8/ADC1_CH7/SUBSPICS1)
- net SPI_nCS_LCD: now also U2.4 (GPIO4/TOUCH4/ADC1_CH3)
- net SPI_nCS_TOUCH: now also U2.5 (GPIO5/TOUCH5/ADC1_CH4)
- net UART0_RX: now also R26.2
- net UART0_TX: now also R25.2
- net VBUS: now also R18.1; no longer C14.1, C15.1, U3.8 (VBUS)
- net at U3.13 (~{RXT}/GPIO.1): now also R29.1
- net at U3.14 (~{TXT}/GPIO.0): now also R28.1
- net at U3.15 (~{SUSPEND}): now also R27.1
- net UART0_nRTS: now reaches U3.19 (~{RTS})
- net UART0_nRTS: now also Q1.2 (E), R24.1
- net at U3.20 (RXD): now also R26.1
- net at U3.21 (TXD): now also R25.1
- net UART0_nDTR: now reaches U3.23 (~{DTR})
- net UART0_nDTR: now also Q2.2 (E), R23.1
- net at U3.9 (~{RST}): now also R20.2
- net JTAG_TCK: now reaches U2.32 (MTCK/GPIO39/CLK_OUT3/SUBSPICS1)
- net JTAG_TDO: now reaches U2.33 (MTDO/GPIO40/CLK_OUT2)
- net JTAG_TDI: now reaches U2.34 (MTDI/GPIO41/CLK_OUT1)
- net JTAG_TMS: now reaches U2.35 (MTMS/GPIO42)
- new net: C13.1, R18.2, R19.1, U3.8 (VBUS)
- new net: D9.1 (K), R29.2
- new net: Q1.1 (B), R23.2
- new net: Q1.3 (C), R30.2
- new net: Q2.1 (B), R24.2
- new net: Q2.3 (C), R31.2
- new net: D8.1 (K), R28.2
- no-connect marks 3 -> 20
Other:
- note added: "USB to UART and automatic reset circuit"
- moved on the sheet: C11, C12, C14, C15, C7, C8, C9, R17, R21, R22, SW1, SW2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

Commit message: schematic, pcb layout, added mouser shoping cart
Parts:
- Q1, Q2: footprint Package_TO_SOT_SMD:SOT-23 -> Package_TO_SOT_SMD:SOT-323_SC-70
