File: Hardware/100008_hw-vern-aqm/100008_hw-vern-aqm.kicad_pcb (KiCad board)
At the start: 2 copper layers, 98 x 56.3 mm, 82 parts, among them J1 Conn_01x14_Socket, J2 USB4220-03-1000-C, J3 Conn_01x06_MountingPin, J4 Conn_01x03_Pin, J5 Conn_01x06_Socket, J6 Conn_01x04_Socket, J7 Conn_01x05_Pin, J8 Conn_01x04_MountingPin, Q1 BC817, Q2 BC817, SW1 SW_Push, SW2 SW_Push, U1 AMS1117-3.3, U2 ESP32-S3-WROOM-1, U3 CP2102N-Axx-xQFN24, U4 SCD40-D-R2, U5 DPS368

Commit message: schematic release, pcb release
Connections:
- net Net-(U2-GPIO19/U1RTS/ADC2_CH8/CLK_OUT2/USB_D-) renamed /Project Architecture/MCU - ESP32/D-
- net Net-(U2-GPIO20/U1CTS/ADC2_CH9/CLK_OUT1/USB_D+) renamed /Project Architecture/MCU - ESP32/D+
Routing:
- net /Project Architecture/MCU - ESP32/D-: track 62.0 -> 59.3 mm
- net /Project Architecture/MCU - ESP32/D+: track 55.2 -> 53.0 mm
- net USB_D-: track 39.7 -> 39.1 mm
- net GND: vias 574 -> 580
- added copper zone on In1.Cu, net GND
- added copper zone on In2.Cu, net GND
Other:
- copper layers 2 -> 4
- rule pad_to_mask_clearance: 0.05 -> 0
