File: Hardware/100008_hw-vern-aqm/Revision History.kicad_sch (KiCad schematic)
At the start: 0 parts

Commit message: schematic release, pcb release
Changed lines of the file:
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@@
 		)
 	)
-	(text_box "- _________________________________\n\n- _________________________________\n\n- _________________________________\n\n- _________________________________\n\n- _________________________________\n\n- _________________________________\n\n- _________________________________\n\n- _________________________________\n\n- _________________________________\n\n- _________________________________\n\n- _________________________________\n\n- _________________________________\n\n- _________________________________\n\n- _________________________________\n\n- _________________________________\n\n- _________________________________\n\n- _________________________________"
+	(text_box "- First prototype release.\n\n- _________________________________\n\n- _________________________________\n\n- _________________________________\n\n- _________________________________\n\n- _________________________________\n\n- _________________________________\n\n- _________________________________\n\n- _________________________________\n\n- _________________________________\n\n- _________________________________\n\n- _________________________________\n\n- _________________________________\n\n- _________________________________\n\n- _________________________________\n\n- _________________________________\n\n- _________________________________"
 		(exclude_from_sim no)
 		(at 22.86 40.64 0)
@@
 		)
 	)
-	(text_box "DD.MM.YYYY - xxx Revision\nVariant: xxx"
+	(text_box "11.11.2024 - Initial Release\nVariant: Rev 10 Prototype"
 		(exclude_from_sim no)
 		(at 20.32 31.75 0)
